Commit message: completed g

File: body.urdf (robot description, URDF)
Before this commit: robot robot, 3 links, 2 joints
Links:
- removed link Link0
- removed link Link1
- removed link Link2
- added link BackLeg, mass 1; collision box size=1 1 1; visual box size=1 1 1
- added link FrontLeg, mass 1; collision box size=1 1 1; visual box size=1 1 1
- added link Torso, mass 1; collision box size=1 1 1; visual box size=1 1 1
Joints:
- removed joint Link0_Link1
- removed joint Link1_Link2
- added joint BackLeg_Torso: type revolute, parent BackLeg, child Torso, origin xyz=1 0 1 rpy=0 0 0, axis 0 1 0, limit lower=-3.14159 upper=3.14159 effort=0.0 velocity=0.0
- added joint Torso_FrontLeg: type revolute, parent Torso, child FrontLeg, origin xyz=1 0 0 rpy=0 0 0, axis 0 1 0, limit lower=-3.14159 upper=3.14159 effort=0.0 velocity=0.0

Commit message: completed n

File: body.urdf (robot description, URDF)
Before this commit: robot robot, 3 links, 2 joints
Links:
- added link LeftLeg, mass 1; collision box size=1 0.2 0.2; visual box size=1 0.2 0.2
- added link RightLeg, mass 1; collision box size=1.0 0.2 0.2; visual box size=1.0 0.2 0.2
- added link lowerBackLeg, mass 1; collision box size=0.2 0.2 1; visual box size=0.2 0.2 1
- added link lowerFrontLeg, mass 1; collision box size=0.2 0.2 1; visual box size=0.2 0.2 1
- added link lowerLeftLeg, mass 1; collision box size=0.2 0.2 1; visual box size=0.2 0.2 1
- added link lowerRightLeg, mass 1; collision box size=0.2 0.2 1; visual box size=0.2 0.2 1
- link BackLeg: geometry collision box size=0.2 1 0.2; visual box size=0.2 1 0.2
- link FrontLeg: geometry collision box size=0.2 1 0.2; visual box size=0.2 1 0.2
Joints:
- added joint BackLeg_lowerBackLeg: type revolute, parent BackLeg, child lowerBackLeg, origin xyz=0 -1 0 rpy=0 0 0, axis 1 0 0, limit lower=-3.14159 upper=3.14159 effort=0.0 velocity=0.0
- added joint FrontLeg_lowerFrontLeg: type revolute, parent FrontLeg, child lowerFrontLeg, origin xyz=0 1 0 rpy=0 0 0, axis 1 0 0, limit lower=-3.14159 upper=3.14159 effort=0.0 velocity=0.0
- added joint LeftLeg_lowerLeftLeg: type revolute, parent LeftLeg, child lowerLeftLeg, origin xyz=-1 0 0 rpy=0 0 0, axis 0 1 0, limit lower=-3.14159 upper=3.14159 effort=0.0 velocity=0.0
- added joint RightLeg_lowerRightLeg: type revolute, parent RightLeg, child lowerRightLeg, origin xyz=1 0 0 rpy=0 0 0, axis 0 1 0, limit lower=-3.14159 upper=3.14159 effort=0.0 velocity=0.0
- added joint Torso_LeftLeg: type revolute, parent Torso, child LeftLeg, origin xyz=-0.5 0 1 rpy=0 0 0, axis 0 1 0, limit lower=-3.14159 upper=3.14159 effort=0.0 velocity=0.0
- added joint Torso_RightLeg: type revolute, parent Torso, child RightLeg, origin xyz=0.5 0 1 rpy=0 0 0, axis 0 1 0, limit lower=-3.14159 upper=3.14159 effort=0.0 velocity=0.0
- joint Torso_BackLeg: axis 0 1 0 -> 1 0 0; origin xyz=1 0 1 rpy=0 0 0 -> xyz=0 -0.5 1 rpy=0 0 0
- joint Torso_FrontLeg: axis 0 1 0 -> 1 0 0; origin xyz=2 0 1 rpy=0 0 0 -> xyz=0 0.5 1 rpy=0 0 0

Commit message: kind of pronks

File: body.urdf (robot description, URDF)
Before this commit: robot robot, 9 links, 8 joints
Links:
- removed link BackLeg
- removed link FrontLeg
- removed link LeftLeg
- removed link RightLeg
- removed link Torso
- removed link lowerBackLeg
- removed link lowerFrontLeg
- removed link lowerLeftLeg
- removed link lowerRightLeg
- added link FrontLeft, mass 1; collision box size=0.2 0.2 3; visual box size=0.2 0.2 3
- added link FrontRight, mass 1; collision box size=0.2 0.2 3; visual box size=0.2 0.2 3
- added link HindLeft, mass 1; collision box size=0.2 0.2 3; visual box size=0.2 0.2 3
- added link HindRight, mass 1; collision box size=0.2 0.2 3; visual box size=0.2 0.2 3
- added link TorsoBack, mass 1; collision box size=2 1 1; visual box size=2 1 1
- added link TorsoFront, mass 1; collision box size=2 1 1; visual box size=2 1 1
Joints:
- removed joint BackLeg_lowerBackLeg
- removed joint FrontLeg_lowerFrontLeg
- removed joint LeftLeg_lowerLeftLeg
- removed joint RightLeg_lowerRightLeg
- removed joint Torso_BackLeg
- removed joint Torso_FrontLeg
- removed joint Torso_LeftLeg
- removed joint Torso_RightLeg
- added joint TorsoBack_HindLeft: type revolute, parent TorsoBack, child HindLeft, origin xyz=-2 0.5 0 rpy=0 0 0, axis 0 1 0, limit lower=-3.14159 upper=3.14159 effort=0.0 velocity=0.0
- added joint TorsoBack_HindRight: type revolute, parent TorsoBack, child HindRight, origin xyz=-2 -0.5 0 rpy=0 0 0, axis 0 1 0, limit lower=-3.14159 upper=3.14159 effort=0.0 velocity=0.0
- added joint TorsoFront_FrontLeft: type revolute, parent TorsoFront, child FrontLeft, origin xyz=3 -0.5 2.5 rpy=0 0 0, axis 0 1 0, limit lower=-3.14159 upper=3.14159 effort=0.0 velocity=0.0
- added joint TorsoFront_FrontRight: type revolute, parent TorsoFront, child FrontRight, origin xyz=3 0.5 2.5 rpy=0 0 0, axis 0 1 0, limit lower=-3.14159 upper=3.14159 effort=0.0 velocity=0.0
- added joint TorsoFront_TorsoBack: type revolute, parent TorsoFront, child TorsoBack, origin xyz=2 0 3.5 rpy=0 0 0, axis 0 1 0, limit lower=-3.14159 upper=3.14159 effort=0.0 velocity=0.0

Commit message: completed assignment 6

File: body.urdf (robot description, URDF)
Before this commit: robot robot, 3 links, 2 joints
Links:
- removed link BackLeg
- removed link FrontLeg
- removed link Torso
- added link 0, mass 1; collision box size=1.5 2.2 1.4; visual box size=1.5 2.2 1.4
- added link 1, mass 1; collision box size=2.8 1.3 1.4; visual box size=2.8 1.3 1.4
- added link 2, mass 1; collision box size=1.1 1.3 2.4; visual box size=1.1 1.3 2.4
- added link 3, mass 1; collision box size=1.9 1.4 2.5; visual box size=1.9 1.4 2.5
- added link 4, mass 1; collision box size=1.5 2.9 2.9; visual box size=1.5 2.9 2.9
- added link 5, mass 1; collision box size=1.6 2.1 2.7; visual box size=1.6 2.1 2.7
- added link 6, mass 1; collision box size=1.9 1.3 2.8; visual box size=1.9 1.3 2.8
- added link 7, mass 1; collision box size=1.3 2.4 2.3; visual box size=1.3 2.4 2.3
Joints:
- removed joint Torso_BackLeg
- removed joint Torso_FrontLeg
- added joint 0_1: type revolute, parent 0, child 1, origin xyz=0.75 0 0.7 rpy=0 0 0, axis 0 1 0, limit lower=-3.14159 upper=3.14159 effort=0.0 velocity=0.0
- added joint 1_2: type revolute, parent 1, child 2, origin xyz=2.8 0 0 rpy=0 0 0, axis 0 1 0, limit lower=-3.14159 upper=3.14159 effort=0.0 velocity=0.0
- added joint 2_3: type revolute, parent 2, child 3, origin xyz=1.1 0 0 rpy=0 0 0, axis 0 1 0, limit lower=-3.14159 upper=3.14159 effort=0.0 velocity=0.0
- added joint 3_4: type revolute, parent 3, child 4, origin xyz=1.9 0 0 rpy=0 0 0, axis 0 1 0, limit lower=-3.14159 upper=3.14159 effort=0.0 velocity=0.0
- added joint 4_5: type revolute, parent 4, child 5, origin xyz=1.5 0 0 rpy=0 0 0, axis 0 1 0, limit lower=-3.14159 upper=3.14159 effort=0.0 velocity=0.0
- added joint 5_6: type revolute, parent 5, child 6, origin xyz=1.6 0 0 rpy=0 0 0, axis 0 1 0, limit lower=-3.14159 upper=3.14159 effort=0.0 velocity=0.0
- added joint 6_7: type revolute, parent 6, child 7, origin xyz=1.9 0 0 rpy=0 0 0, axis 0 1 0, limit lower=-3.14159 upper=3.14159 effort=0.0 velocity=0.0

Commit message: completed snake1d phc

File: body.urdf (robot description, URDF)
Before this commit: robot robot, 3 links, 2 joints
Links:
- removed link BackLeg
- removed link FrontLeg
- removed link Torso
- added link 0, mass 1; collision box size=1.1 1.8 1.5; visual box size=1.1 1.8 1.5
- added link 1, mass 1; collision box size=1.5 1.7 3.0; visual box size=1.5 1.7 3.0
- added link 2, mass 1; collision box size=1.8 2.6 1.3; visual box size=1.8 2.6 1.3
Joints:
- removed joint Torso_BackLeg
- removed joint Torso_FrontLeg
- added joint 0_1: type revolute, parent 0, child 1, origin xyz=0.55 0 0.75 rpy=0 0 0, axis 0 1 0, limit lower=-3.14159 upper=3.14159 effort=0.0 velocity=0.0
- added joint 1_2: type revolute, parent 1, child 2, origin xyz=1.5 0 0 rpy=0 0 0, axis 0 1 0, limit lower=-3.14159 upper=3.14159 effort=0.0 velocity=0.0

Commit message: 3d concept done need axis

File: body.urdf (robot description, URDF)
Before this commit: robot robot, 3 links, 2 joints
Links:
- added link 3, mass 1; collision box size=1.7 1.3 1.6; visual box size=1.7 1.3 1.6
- added link 4, mass 1; collision box size=2.5 3.0 1.8; visual box size=2.5 3.0 1.8
- added link 5, mass 1; collision box size=2.6 1.8 2.9; visual box size=2.6 1.8 2.9
- added link 6, mass 1; collision box size=2.6 1.5 1.4; visual box size=2.6 1.5 1.4
- link 0: geometry collision box size=2.8 2.6 1.4; visual box size=2.8 2.6 1.4
- link 1: geometry collision box size=1.9 1.0 2.0; visual box size=1.9 1.0 2.0
- link 2: geometry collision box size=1.4 2.2 2.2; visual box size=1.4 2.2 2.2
Joints:
- added joint 2_3: type revolute, parent 2, child 3, origin xyz=0.7 0 1.1 rpy=0 0 0, axis 0 1 0, limit lower=-3.14159 upper=3.14159 effort=0.0 velocity=0.0
- added joint 3_4: type revolute, parent 3, child 4, origin xyz=0.85 0 0.8 rpy=0 0 0, axis 0 1 0, limit lower=-3.14159 upper=3.14159 effort=0.0 velocity=0.0
- added joint 4_5: type revolute, parent 4, child 5, origin xyz=1.25 0 0.9 rpy=0 0 0, axis 0 1 0, limit lower=-3.14159 upper=3.14159 effort=0.0 velocity=0.0
- added joint 5_6: type revolute, parent 5, child 6, origin xyz=1.3 0 1.45 rpy=0 0 0, axis 0 1 0, limit lower=-3.14159 upper=3.14159 effort=0.0 velocity=0.0
- joint 0_1: origin xyz=0.55 0 0.75 rpy=0 0 0 -> xyz=1.4 0 0.7 rpy=0 0 0
- joint 1_2: origin xyz=1.5 0 0 rpy=0 0 0 -> xyz=0.95 0 1.0 rpy=0 0 0

Commit message: completed snake3d

File: body.urdf (robot description, URDF)
Before this commit: robot robot, 7 links, 6 joints
Links:
- link 0: geometry collision box size=1.2 2.0 1.0; visual box size=1.2 2.0 1.0
- link 1: geometry collision box size=1.9 0.9 0.7; visual box size=1.9 0.9 0.7
- link 2: geometry collision box size=0.6 1.7 0.7; visual box size=0.6 1.7 0.7
- link 3: geometry collision box size=1.1 1.3 0.7; visual box size=1.1 1.3 0.7
- link 4: geometry collision box size=0.4 1.8 0.9; visual box size=0.4 1.8 0.9
- link 5: geometry collision box size=1.9 1.8 1.4; visual box size=1.9 1.8 1.4
- link 6: geometry collision box size=1.4 0.8 0.3; visual box size=1.4 0.8 0.3
Joints:
- joint 0_1: origin xyz=1.4 0 0.7 rpy=0 0 0 -> xyz=0.6 0 0.5 rpy=0 0 0
- joint 1_2: axis 0 1 0 -> 0 0 1; origin xyz=0.95 0 1.0 rpy=0 0 0 -> xyz=0.95 0.45 0 rpy=0 0 0
- joint 2_3: axis 0 1 0 -> 1 0 0; origin xyz=0.7 0 1.1 rpy=0 0 0 -> xyz=0 0.85 0.35 rpy=0 0 0
- joint 3_4: axis 0 1 0 -> 0 0 1; origin xyz=0.85 0 0.8 rpy=0 0 0 -> xyz=0 0 0.7 rpy=0 0 0
- joint 4_5: axis 0 1 0 -> 1 0 0; origin xyz=1.25 0 0.9 rpy=0 0 0 -> xyz=0 0.9 0.45 rpy=0 0 0
- joint 5_6: axis 0 1 0 -> 1 0 0; origin xyz=1.3 0 1.45 rpy=0 0 0 -> xyz=0 0.9 0.7 rpy=0 0 0

Commit message: done

File: body.urdf (robot description, URDF)
Before this commit: robot robot, 8 links, 7 joints
Links:
- added link 8, mass 1; collision box size=2.1 2.9 2.4; visual box size=2.1 2.9 2.4
- added link 9, mass 1; collision box size=2.1 1.9 1.8; visual box size=2.1 1.9 1.8
- link 0: geometry collision box size=1.8 2.1 2.6; visual box size=1.8 2.1 2.6
- link 1: geometry collision box size=2.0 3.0 1.2; visual box size=2.0 3.0 1.2
- link 2: geometry collision box size=1.6 2.6 1.8; visual box size=1.6 2.6 1.8
- link 3: geometry collision box size=2.7 1.5 3.0; visual box size=2.7 1.5 3.0
- link 4: geometry collision box size=1.0 1.2 2.9; visual box size=1.0 1.2 2.9
- link 5: geometry collision box size=1.0 2.4 2.0; visual box size=1.0 2.4 2.0
- link 6: geometry collision box size=1.9 1.4 1.2; visual box size=1.9 1.4 1.2
- link 7: geometry collision box size=1.6 1.8 1.3; visual box size=1.6 1.8 1.3
Joints:
- added joint 7_8: type revolute, parent 7, child 8, origin xyz=1.6 0 0 rpy=0 0 0, axis 0 1 0, limit lower=-3.14159 upper=3.14159 effort=0.0 velocity=0.0
- added joint 8_9: type revolute, parent 8, child 9, origin xyz=2.1 0 0 rpy=0 0 0, axis 0 1 0, limit lower=-3.14159 upper=3.14159 effort=0.0 velocity=0.0
- joint 0_1: origin xyz=0.75 0 0.7 rpy=0 0 0 -> xyz=0.9 0 1.3 rpy=0 0 0
- joint 1_2: origin xyz=2.8 0 0 rpy=0 0 0 -> xyz=2.0 0 0 rpy=0 0 0
- joint 2_3: origin xyz=1.1 0 0 rpy=0 0 0 -> xyz=1.6 0 0 rpy=0 0 0
- joint 3_4: origin xyz=1.9 0 0 rpy=0 0 0 -> xyz=2.7 0 0 rpy=0 0 0
- joint 4_5: origin xyz=1.5 0 0 rpy=0 0 0 -> xyz=1.0 0 0 rpy=0 0 0
- joint 5_6: origin xyz=1.6 0 0 rpy=0 0 0 -> xyz=1.0 0 0 rpy=0 0 0

Commit message: done

File: body.urdf (robot description, URDF)
Before this commit: robot robot, 3 links, 2 joints
Links:
- added link 3, mass 1; collision box size=1.3 1.5 2.8; visual box size=1.3 1.5 2.8
- added link 4, mass 1; collision box size=2.2 2.5 2.1; visual box size=2.2 2.5 2.1
- added link 5, mass 1; collision box size=1.4 2.4 2.4; visual box size=1.4 2.4 2.4
- added link 6, mass 1; collision box size=2.0 2.0 1.1; visual box size=2.0 2.0 1.1
- link 0: geometry collision box size=2.3 2.7 1.7; visual box size=2.3 2.7 1.7
- link 1: geometry collision box size=2.0 2.1 1.1; visual box size=2.0 2.1 1.1
- link 2: geometry collision box size=1.2 1.6 2.0; visual box size=1.2 1.6 2.0
Joints:
- added joint 2_3: type revolute, parent 2, child 3, origin xyz=1.2 0 0 rpy=0 0 0, axis 0 1 0, limit lower=-3.14159 upper=3.14159 effort=0.0 velocity=0.0
- added joint 3_4: type revolute, parent 3, child 4, origin xyz=1.3 0 0 rpy=0 0 0, axis 0 1 0, limit lower=-3.14159 upper=3.14159 effort=0.0 velocity=0.0
- added joint 4_5: type revolute, parent 4, child 5, origin xyz=2.2 0 0 rpy=0 0 0, axis 0 1 0, limit lower=-3.14159 upper=3.14159 effort=0.0 velocity=0.0
- added joint 5_6: type revolute, parent 5, child 6, origin xyz=1.4 0 0 rpy=0 0 0, axis 0 1 0, limit lower=-3.14159 upper=3.14159 effort=0.0 velocity=0.0
- joint 0_1: origin xyz=0.55 0 0.75 rpy=0 0 0 -> xyz=1.15 0 0.85 rpy=0 0 0
- joint 1_2: origin xyz=1.5 0 0 rpy=0 0 0 -> xyz=2.0 0 0 rpy=0 0 0

Commit message: done

File: body.urdf (robot description, URDF)
Before this commit: robot robot, 10 links, 9 joints
Links:
- added link 10, mass 1; collision box size=2.6 2.9 2.9; visual box size=2.6 2.9 2.9
- added link 11, mass 1; collision box size=2.5 1.3 1.5; visual box size=2.5 1.3 1.5
- added link 12, mass 1; collision box size=2.7 1.7 1.3; visual box size=2.7 1.7 1.3
- link 0: geometry collision box size=1.1 1.5 2.2; visual box size=1.1 1.5 2.2
- link 1: geometry collision box size=2.5 2.5 2.1; visual box size=2.5 2.5 2.1
- link 2: geometry collision box size=1.0 2.6 2.4; visual box size=1.0 2.6 2.4
- link 3: geometry collision box size=1.1 3.0 2.8; visual box size=1.1 3.0 2.8
- link 4: geometry collision box size=2.7 2.6 2.0; visual box size=2.7 2.6 2.0
- link 5: geometry collision box size=1.2 2.8 1.1; visual box size=1.2 2.8 1.1
- link 6: geometry collision box size=1.3 1.3 1.0; visual box size=1.3 1.3 1.0
- link 7: geometry collision box size=2.1 1.4 1.2; visual box size=2.1 1.4 1.2
- link 8: geometry collision box size=1.3 2.9 2.9; visual box size=1.3 2.9 2.9
- link 9: geometry collision box size=2.5 1.4 2.3; visual box size=2.5 1.4 2.3
Joints:
- added joint 10_11: type revolute, parent 10, child 11, origin xyz=2.6 0 0 rpy=0 0 0, axis 0 1 0, limit lower=-3.14159 upper=3.14159 effort=0.0 velocity=0.0
- added joint 11_12: type revolute, parent 11, child 12, origin xyz=2.5 0 0 rpy=0 0 0, axis 0 1 0, limit lower=-3.14159 upper=3.14159 effort=0.0 velocity=0.0
- added joint 9_10: type revolute, parent 9, child 10, origin xyz=2.5 0 0 rpy=0 0 0, axis 0 1 0, limit lower=-3.14159 upper=3.14159 effort=0.0 velocity=0.0
- joint 0_1: origin xyz=0.9 0 1.3 rpy=0 0 0 -> xyz=0.55 0 1.1 rpy=0 0 0
- joint 1_2: origin xyz=2.0 0 0 rpy=0 0 0 -> xyz=2.5 0 0 rpy=0 0 0
- joint 2_3: origin xyz=1.6 0 0 rpy=0 0 0 -> xyz=1.0 0 0 rpy=0 0 0
- joint 3_4: origin xyz=2.7 0 0 rpy=0 0 0 -> xyz=1.1 0 0 rpy=0 0 0
- joint 4_5: origin xyz=1.0 0 0 rpy=0 0 0 -> xyz=2.7 0 0 rpy=0 0 0
- joint 5_6: origin xyz=1.0 0 0 rpy=0 0 0 -> xyz=1.2 0 0 rpy=0 0 0
- joint 6_7: origin xyz=1.9 0 0 rpy=0 0 0 -> xyz=1.3 0 0 rpy=0 0 0
- joint 7_8: origin xyz=1.6 0 0 rpy=0 0 0 -> xyz=2.1 0 0 rpy=0 0 0
- joint 8_9: origin xyz=2.1 0 0 rpy=0 0 0 -> xyz=1.3 0 0 rpy=0 0 0

Commit message: s

File: body.urdf (robot description, URDF)
Before this commit: robot robot, 7 links, 6 joints
Links:
- link 0: geometry collision box size=0.9 1.8 0.4; visual box size=0.9 1.8 0.4
- link 1: geometry collision box size=1.9 0.4 2.0; visual box size=1.9 0.4 2.0
- link 2: geometry collision box size=1.5 0.4 1.4; visual box size=1.5 0.4 1.4
- link 3: geometry collision box size=0.5 1.4 1.3; visual box size=0.5 1.4 1.3
- link 4: geometry collision box size=0.6 0.2 0.7; visual box size=0.6 0.2 0.7
- link 5: geometry collision box size=1.4 1.3 1.8; visual box size=1.4 1.3 1.8
- link 6: geometry collision box size=1.8 1.7 0.7; visual box size=1.8 1.7 0.7
Joints:
- joint 0_1: origin xyz=0.6 0 0.5 rpy=0 0 0 -> xyz=0.45 0 0.2 rpy=0 0 0
- joint 1_2: axis 0 0 1 -> 0 1 0; origin xyz=0.95 0.45 0 rpy=0 0 0 -> xyz=0.95 0 1.0 rpy=0 0 0
- joint 2_3: axis 1 0 0 -> 0 0 1; origin xyz=0 0.85 0.35 rpy=0 0 0 -> xyz=0 0 1.4 rpy=0 0 0
- joint 3_4: origin xyz=0 0 0.7 rpy=0 0 0 -> xyz=0 0 1.3 rpy=0 0 0
- joint 4_5: origin xyz=0 0.9 0.45 rpy=0 0 0 -> xyz=0.3 0 0.35 rpy=0 0 0
- joint 5_6: axis 1 0 0 -> 0 0 1; origin xyz=0 0.9 0.7 rpy=0 0 0 -> xyz=0.7 0 0.9 rpy=0 0 0

Commit message: colors

File: body.urdf (robot description, URDF)
Before this commit: robot robot, 7 links, 6 joints
Links:
- link 0: geometry collision box size=1.7 1.0 2.0; visual box size=1.7 1.0 2.0
- link 1: geometry collision box size=1.9 0.7 1.9; visual box size=1.9 0.7 1.9
- link 2: geometry collision box size=1.8 0.4 0.5; visual box size=1.8 0.4 0.5
- link 3: geometry collision box size=1.2 1.9 1.9; visual box size=1.2 1.9 1.9
- link 4: geometry collision box size=1.0 0.7 0.5; visual box size=1.0 0.7 0.5
- link 5: geometry collision box size=0.2 0.3 0.3; visual box size=0.2 0.3 0.3
- link 6: geometry collision box size=0.7 1.6 0.6; visual box size=0.7 1.6 0.6
Joints:
- joint 0_1: origin xyz=0.45 0 0.2 rpy=0 0 0 -> xyz=0.85 0 1.0 rpy=0 0 0
- joint 1_2: origin xyz=0.95 0 1.0 rpy=0 0 0 -> xyz=1.9 0 0 rpy=0 0 0
- joint 2_3: origin xyz=0 0 1.4 rpy=0 0 0 -> xyz=0.9 0.2 0 rpy=0 0 0
- joint 3_4: axis 0 0 1 -> 1 0 0; origin xyz=0 0 1.3 rpy=0 0 0 -> xyz=0 1.9 0 rpy=0 0 0
- joint 4_5: origin xyz=0.3 0 0.35 rpy=0 0 0 -> xyz=0.5 0.35 0 rpy=0 0 0
- joint 5_6: axis 0 0 1 -> 1 0 0; origin xyz=0.7 0 0.9 rpy=0 0 0 -> xyz=0.1 0.15 0 rpy=0 0 0

Commit message: cancer

File: body.urdf (robot description, URDF)
Before this commit: robot robot, 7 links, 6 joints
Links:
- link 0: geometry collision box size=0.9 0.6 0.8; visual box size=0.9 0.6 0.8
- link 1: geometry collision box size=1.0 0.7 0.8; visual box size=1.0 0.7 0.8
- link 2: geometry collision box size=0.9 0.5 0.5; visual box size=0.9 0.5 0.5
- link 3: geometry collision box size=1.0 0.7 0.7; visual box size=1.0 0.7 0.7
- link 4: geometry collision box size=0.7 0.7 0.6; visual box size=0.7 0.7 0.6
- link 5: geometry collision box size=0.8 0.9 0.6; visual box size=0.8 0.9 0.6
- link 6: geometry collision box size=0.7 0.8 0.8; visual box size=0.7 0.8 0.8
Joints:
- joint 0_1: origin xyz=0.85 0 1.0 rpy=0 0 0 -> xyz=0.45 0 0.4 rpy=0 0 0
- joint 1_2: axis 0 1 0 -> 0 0 1; origin xyz=1.9 0 0 rpy=0 0 0 -> xyz=1.0 0 0 rpy=0 0 0
- joint 2_3: axis 0 0 1 -> 1 0 0; origin xyz=0.9 0.2 0 rpy=0 0 0 -> xyz=0.45 0 0.25 rpy=0 0 0
- joint 3_4: origin xyz=0 1.9 0 rpy=0 0 0 -> xyz=0.5 0 0.35 rpy=0 0 0
- joint 4_5: origin xyz=0.5 0.35 0 rpy=0 0 0 -> xyz=0.35 0.35 0 rpy=0 0 0
- joint 5_6: origin xyz=0.1 0.15 0 rpy=0 0 0 -> xyz=0 0.9 0 rpy=0 0 0

Commit message: wow

File: body.urdf (robot description, URDF)
Before this commit: robot robot, 7 links, 6 joints
Links:
- removed link 6
- link 0: geometry collision box size=0.9 0.6 0.7; visual box size=0.9 0.6 0.7
- link 1: geometry collision box size=0.8 0.9 0.6; visual box size=0.8 0.9 0.6
- link 2: geometry collision box size=0.8 0.6 1.0; visual box size=0.8 0.6 1.0
- link 3: geometry collision box size=0.5 0.8 0.7; visual box size=0.5 0.8 0.7
- link 4: geometry collision box size=0.9 0.6 0.7; visual box size=0.9 0.6 0.7
- link 5: geometry collision box size=0.8 0.8 0.5; visual box size=0.8 0.8 0.5
Joints:
- removed joint 4_5
- removed joint 5_6
- added joint 1_5: type revolute, parent 1, child 5, origin xyz=0 0.45 0.6 rpy=0 0 0, axis 1 0 0, limit lower=-3.14159 upper=3.14159 effort=0.0 velocity=0.0
- joint 0_1: axis 0 1 0 -> 0 0 1; origin xyz=0.45 0 0.4 rpy=0 0 0 -> xyz=0 0 0.7 rpy=0 0 0
- joint 1_2: origin xyz=1.0 0 0 rpy=0 0 0 -> xyz=0 0 0.6 rpy=0 0 0
- joint 2_3: axis 1 0 0 -> 0 0 1; origin xyz=0.45 0 0.25 rpy=0 0 0 -> xyz=0.4 0 0.5 rpy=0 0 0
- joint 3_4: origin xyz=0.5 0 0.35 rpy=0 0 0 -> xyz=0.5 0 0 rpy=0 0 0

Commit message: a7

File: body.urdf (robot description, URDF)
Before this commit: robot robot, 6 links, 5 joints
Links:
- added link 6, mass 1; collision box size=0.9 0.5 0.7; visual box size=0.9 0.5 0.7
- link 0: geometry collision box size=1.0 0.9 0.5; visual box size=1.0 0.9 0.5
- link 1: geometry collision box size=0.7 1.0 0.7; visual box size=0.7 1.0 0.7
- link 2: geometry collision box size=0.6 0.9 1.0; visual box size=0.6 0.9 1.0
- link 3: geometry collision box size=0.6 0.8 0.5; visual box size=0.6 0.8 0.5
- link 4: geometry collision box size=0.5 0.8 1.0; visual box size=0.5 0.8 1.0
- link 5: geometry collision box size=0.9 0.5 0.6; visual box size=0.9 0.5 0.6
Joints:
- removed joint 1_5
- removed joint 3_4
- added joint 1_4: type revolute, parent 1, child 4, origin xyz=0.7 0.5 0 rpy=0 0 0, axis 1 0 0, limit lower=-3.14159 upper=3.14159 effort=0.0 velocity=0.0
- added joint 4_5: type revolute, parent 4, child 5, origin xyz=0 0.4 0.5 rpy=0 0 0, axis 0 1 0, limit lower=-3.14159 upper=3.14159 effort=0.0 velocity=0.0
- added joint 4_6: type revolute, parent 4, child 6, origin xyz=0 0.4 1.0 rpy=0 0 0, axis 0 1 0, limit lower=-3.14159 upper=3.14159 effort=0.0 velocity=0.0
- joint 0_1: axis 0 0 1 -> 0 1 0; origin xyz=0 0 0.7 rpy=0 0 0 -> xyz=0.5 0 0.25 rpy=0 0 0
- joint 1_2: axis 0 0 1 -> 0 1 0; origin xyz=0 0 0.6 rpy=0 0 0 -> xyz=0.7 0 0 rpy=0 0 0
- joint 2_3: axis 0 0 1 -> 0 1 0; origin xyz=0.4 0 0.5 rpy=0 0 0 -> xyz=0.6 0 0 rpy=0 0 0
