Commit message: 857

File: body.urdf (robot description, URDF)
Before this commit: robot robot, 7 links, 6 joints
Links:
- removed link 6
- link 0: geometry collision box size=0.7 0.5 0.8; visual box size=0.7 0.5 0.8
- link 1: geometry collision box size=0.5 0.7 0.8; visual box size=0.5 0.7 0.8
- link 2: geometry collision box size=0.7 1.0 0.7; visual box size=0.7 1.0 0.7
- link 3: geometry collision box size=1.0 0.6 0.7; visual box size=1.0 0.6 0.7
- link 4: geometry collision box size=0.9 0.7 0.7; visual box size=0.9 0.7 0.7
- link 5: geometry collision box size=0.9 0.5 0.9; visual box size=0.9 0.5 0.9
Joints:
- removed joint 1_2
- removed joint 1_4
- removed joint 4_5
- removed joint 4_6
- added joint 0_2: type revolute, parent 0, child 2, origin xyz=0.35 0.25 0.4 rpy=0 0 0, axis 0 1 0, limit lower=-3.14159 upper=3.14159 effort=0.0 velocity=0.0
- added joint 1_5: type revolute, parent 1, child 5, origin xyz=0.25 0 0.4 rpy=0 0 0, axis 0 1 0, limit lower=-3.14159 upper=3.14159 effort=0.0 velocity=0.0
- added joint 2_4: type revolute, parent 2, child 4, origin xyz=0.35 1.0 0 rpy=0 0 0, axis 0 0 1, limit lower=-3.14159 upper=3.14159 effort=0.0 velocity=0.0
- joint 0_1: axis 0 1 0 -> 0 0 1; origin xyz=0.5 0 0.25 rpy=0 0 0 -> xyz=0.35 0 0.4 rpy=0 0 0
- joint 2_3: origin xyz=0.6 0 0 rpy=0 0 0 -> xyz=0 1.0 0 rpy=0 0 0
