Commit message: before making genbrain correct

File: body5.urdf (robot description, URDF)
Before this commit: robot robot, 15 links, 14 joints
Links:
- link 0: geometry collision box size=0.6 0.7 0.6; visual box size=0.6 0.7 0.6
- link 1: geometry collision box size=0.9 0.8 0.6; visual box size=0.9 0.8 0.6
- link 10: geometry collision box size=0.8 0.6 1.0; visual box size=0.8 0.6 1.0
- link 11: geometry collision box size=0.9 0.8 0.6; visual box size=0.9 0.8 0.6
- link 12: geometry collision box size=1.0 0.6 0.6; visual box size=1.0 0.6 0.6
- link 13: geometry collision box size=0.5 1.0 0.6; visual box size=0.5 1.0 0.6
- link 14: geometry collision box size=0.9 0.5 0.8; visual box size=0.9 0.5 0.8
- link 2: geometry collision box size=0.7 0.8 0.7; visual box size=0.7 0.8 0.7
- link 3: geometry collision box size=0.9 0.8 0.6; visual box size=0.9 0.8 0.6
- link 4: geometry collision box size=0.6 0.7 0.5; visual box size=0.6 0.7 0.5
- link 5: geometry collision box size=0.9 0.9 0.6; visual box size=0.9 0.9 0.6
- link 6: geometry collision box size=0.8 0.9 0.6; visual box size=0.8 0.9 0.6
- link 7: geometry collision box size=0.7 0.6 0.6; visual box size=0.7 0.6 0.6
- link 8: geometry collision box size=1.0 0.8 0.5; visual box size=1.0 0.8 0.5
- link 9: geometry collision box size=0.9 0.9 0.7; visual box size=0.9 0.9 0.7
Joints:
- removed joint 10_13
- removed joint 1_10
- removed joint 1_4
- removed joint 2_3
- removed joint 2_7
- removed joint 4_8
- removed joint 6_9
- removed joint 7_11
- removed joint 8_12
- removed joint 8_14
- added joint 10_12: type revolute, parent 10, child 12, origin xyz=-0.4 0 0.5 rpy=0 0 0, axis 0 1 0, limit lower=-3.14159 upper=3.14159 effort=0.0 velocity=0.0
- added joint 10_14: type revolute, parent 10, child 14, origin xyz=0 -0.3 0.5 rpy=0 0 0, axis 1 0 0, limit lower=-3.14159 upper=3.14159 effort=0.0 velocity=0.0
- added joint 1_3: type revolute, parent 1, child 3, origin xyz=-0.45 -0.4 0 rpy=0 0 0, axis 0 0 1, limit lower=-3.14159 upper=3.14159 effort=0.0 velocity=0.0
- added joint 1_7: type revolute, parent 1, child 7, origin xyz=0 -0.8 0 rpy=0 0 0, axis 1 0 0, limit lower=-3.14159 upper=3.14159 effort=0.0 velocity=0.0
- added joint 3_4: type revolute, parent 3, child 4, origin xyz=-0.45 0.4 0 rpy=0 0 0, axis 0 1 0, limit lower=-3.14159 upper=3.14159 effort=0.0 velocity=0.0
- added joint 5_9: type revolute, parent 5, child 9, origin xyz=-0.45 -0.45 0 rpy=0 0 0, axis 1 0 0, limit lower=-3.14159 upper=3.14159 effort=0.0 velocity=0.0
- added joint 6_8: type revolute, parent 6, child 8, origin xyz=-0.4 -0.45 0 rpy=0 0 0, axis 1 0 0, limit lower=-3.14159 upper=3.14159 effort=0.0 velocity=0.0
- added joint 8_10: type revolute, parent 8, child 10, origin xyz=-0.5 0 0.25 rpy=0 0 0, axis 0 0 1, limit lower=-3.14159 upper=3.14159 effort=0.0 velocity=0.0
- added joint 8_13: type revolute, parent 8, child 13, origin xyz=-1.0 0 0 rpy=0 0 0, axis 0 0 1, limit lower=-3.14159 upper=3.14159 effort=0.0 velocity=0.0
- added joint 9_11: type revolute, parent 9, child 11, origin xyz=0 -0.9 0 rpy=0 0 0, axis 0 1 0, limit lower=-3.14159 upper=3.14159 effort=0.0 velocity=0.0
- joint 0_1: axis 1 0 0 -> 0 0 1; origin xyz=0 0.4 0.3 rpy=0 0 0 -> xyz=0 -0.35 0.3 rpy=0 0 0
- joint 0_2: axis 1 0 0 -> 0 1 0
- joint 2_5: axis 1 0 0 -> 0 1 0; origin xyz=-0.45 0 0.35 rpy=0 0 0 -> xyz=-0.35 0 0.35 rpy=0 0 0
- joint 3_6: origin xyz=0.3 -0.4 0 rpy=0 0 0 -> xyz=-0.45 -0.4 0 rpy=0 0 0

File: body6.urdf (robot description, URDF)
Before this commit: robot robot, 15 links, 14 joints
Links:
- link 0: geometry collision box size=0.9 0.8 0.7; visual box size=0.9 0.8 0.7
- link 1: geometry collision box size=0.5 0.9 0.9; visual box size=0.5 0.9 0.9
- link 10: geometry collision box size=1.0 0.6 0.7; visual box size=1.0 0.6 0.7
- link 11: geometry collision box size=0.5 0.8 0.9; visual box size=0.5 0.8 0.9
- link 12: geometry collision box size=1.0 1.0 0.8; visual box size=1.0 1.0 0.8
- link 13: geometry collision box size=0.5 0.9 0.6; visual box size=0.5 0.9 0.6
- link 14: geometry collision box size=1.0 0.9 0.8; visual box size=1.0 0.9 0.8
- link 2: geometry collision box size=0.6 0.5 0.7; visual box size=0.6 0.5 0.7
- link 3: geometry collision box size=0.9 0.7 0.5; visual box size=0.9 0.7 0.5
- link 4: geometry collision box size=0.8 0.6 0.6; visual box size=0.8 0.6 0.6
- link 5: geometry collision box size=0.7 0.6 0.6; visual box size=0.7 0.6 0.6
- link 6: geometry collision box size=0.8 0.6 0.5; visual box size=0.8 0.6 0.5
- link 7: geometry collision box size=1.0 0.6 0.9; visual box size=1.0 0.6 0.9
- link 8: geometry collision box size=0.6 0.9 0.8; visual box size=0.6 0.9 0.8
- link 9: geometry collision box size=0.9 0.7 0.6; visual box size=0.9 0.7 0.6
Joints:
- removed joint 1_10
- removed joint 1_4
- removed joint 2_3
- removed joint 2_5
- removed joint 2_7
- removed joint 3_6
- removed joint 4_8
- removed joint 6_9
- removed joint 7_11
- removed joint 8_12
- removed joint 8_14
- added joint 0_3: type revolute, parent 0, child 3, origin xyz=-0.45 0 0.35 rpy=0 0 0, axis 1 0 0, limit lower=-3.14159 upper=3.14159 effort=0.0 velocity=0.0
- added joint 10_12: type revolute, parent 10, child 12, origin xyz=0 0 0.7 rpy=0 0 0, axis 0 1 0, limit lower=-3.14159 upper=3.14159 effort=0.0 velocity=0.0
- added joint 13_14: type revolute, parent 13, child 14, origin xyz=-0.5 0 0 rpy=0 0 0, axis 0 1 0, limit lower=-3.14159 upper=3.14159 effort=0.0 velocity=0.0
- added joint 1_11: type revolute, parent 1, child 11, origin xyz=-0.25 0 0.45 rpy=0 0 0, axis 0 1 0, limit lower=-3.14159 upper=3.14159 effort=0.0 velocity=0.0
- added joint 1_6: type revolute, parent 1, child 6, origin xyz=0.25 0 0.45 rpy=0 0 0, axis 0 0 1, limit lower=-3.14159 upper=3.14159 effort=0.0 velocity=0.0
- added joint 2_4: type revolute, parent 2, child 4, origin xyz=0 -0.5 0 rpy=0 0 0, axis 1 0 0, limit lower=-3.14159 upper=3.14159 effort=0.0 velocity=0.0
- added joint 3_9: type revolute, parent 3, child 9, origin xyz=-0.45 0.35 0 rpy=0 0 0, axis 1 0 0, limit lower=-3.14159 upper=3.14159 effort=0.0 velocity=0.0
- added joint 4_5: type revolute, parent 4, child 5, origin xyz=0 -0.6 0 rpy=0 0 0, axis 0 1 0, limit lower=-3.14159 upper=3.14159 effort=0.0 velocity=0.0
- added joint 4_7: type revolute, parent 4, child 7, origin xyz=0 -0.3 0.3 rpy=0 0 0, axis 0 0 1, limit lower=-3.14159 upper=3.14159 effort=0.0 velocity=0.0
- added joint 7_10: type revolute, parent 7, child 10, origin xyz=0 0 0.9 rpy=0 0 0, axis 0 0 1, limit lower=-3.14159 upper=3.14159 effort=0.0 velocity=0.0
- added joint 7_8: type revolute, parent 7, child 8, origin xyz=-0.5 0 0.45 rpy=0 0 0, axis 0 1 0, limit lower=-3.14159 upper=3.14159 effort=0.0 velocity=0.0
- joint 0_1: axis 1 0 0 -> 0 0 1; origin xyz=0 0.4 0.3 rpy=0 0 0 -> xyz=0 0 0.7 rpy=0 0 0
- joint 0_2: axis 1 0 0 -> 0 0 1; origin xyz=0 0 0.6 rpy=0 0 0 -> xyz=0 -0.4 0.35 rpy=0 0 0
- joint 10_13: axis 0 1 0 -> 0 0 1; origin xyz=-0.3 0 0.4 rpy=0 0 0 -> xyz=-0.5 0 0.35 rpy=0 0 0

File: body7.urdf (robot description, URDF)
Before this commit: robot robot, 15 links, 14 joints
Links:
- link 0: geometry collision box size=0.8 0.7 0.8; visual box size=0.8 0.7 0.8
- link 1: geometry collision box size=0.8 0.8 0.6; visual box size=0.8 0.8 0.6
- link 10: geometry collision box size=0.7 0.7 0.8; visual box size=0.7 0.7 0.8
- link 11: geometry collision box size=0.9 0.9 0.7; visual box size=0.9 0.9 0.7
- link 12: geometry collision box size=0.9 1.0 1.0; visual box size=0.9 1.0 1.0
- link 13: geometry collision box size=0.8 0.9 0.6; visual box size=0.8 0.9 0.6
- link 14: geometry collision box size=0.8 0.6 0.6; visual box size=0.8 0.6 0.6
- link 2: geometry collision box size=0.8 0.9 0.9; visual box size=0.8 0.9 0.9
- link 3: geometry collision box size=0.8 0.7 0.8; visual box size=0.8 0.7 0.8
- link 4: geometry collision box size=0.7 0.7 0.7; visual box size=0.7 0.7 0.7
- link 5: geometry collision box size=0.9 0.5 0.7; visual box size=0.9 0.5 0.7
- link 6: geometry collision box size=0.7 0.7 0.9; visual box size=0.7 0.7 0.9
- link 7: geometry collision box size=0.6 0.7 0.8; visual box size=0.6 0.7 0.8
- link 8: geometry collision box size=0.9 0.6 0.6; visual box size=0.9 0.6 0.6
- link 9: geometry collision box size=0.9 0.7 0.6; visual box size=0.9 0.7 0.6
Joints:
- removed joint 10_13
- removed joint 1_10
- removed joint 1_4
- removed joint 2_3
- removed joint 2_5
- removed joint 2_7
- removed joint 3_6
- removed joint 4_8
- removed joint 6_9
- removed joint 7_11
- removed joint 8_12
- removed joint 8_14
- added joint 11_12: type revolute, parent 11, child 12, origin xyz=0.9 0 0 rpy=0 0 0, axis 0 1 0, limit lower=-3.14159 upper=3.14159 effort=0.0 velocity=0.0
- added joint 1_3: type revolute, parent 1, child 3, origin xyz=-0.8 0 0 rpy=0 0 0, axis 1 0 0, limit lower=-3.14159 upper=3.14159 effort=0.0 velocity=0.0
- added joint 1_5: type revolute, parent 1, child 5, origin xyz=-0.4 -0.4 0 rpy=0 0 0, axis 1 0 0, limit lower=-3.14159 upper=3.14159 effort=0.0 velocity=0.0
- added joint 2_14: type revolute, parent 2, child 14, origin xyz=0.4 0 0.45 rpy=0 0 0, axis 1 0 0, limit lower=-3.14159 upper=3.14159 effort=0.0 velocity=0.0
- added joint 2_8: type revolute, parent 2, child 8, origin xyz=0 0 0.9 rpy=0 0 0, axis 0 0 1, limit lower=-3.14159 upper=3.14159 effort=0.0 velocity=0.0
- added joint 2_9: type revolute, parent 2, child 9, origin xyz=0 -0.45 0.45 rpy=0 0 0, axis 0 0 1, limit lower=-3.14159 upper=3.14159 effort=0.0 velocity=0.0
- added joint 3_4: type revolute, parent 3, child 4, origin xyz=-0.4 0.35 0 rpy=0 0 0, axis 0 0 1, limit lower=-3.14159 upper=3.14159 effort=0.0 velocity=0.0
- added joint 3_7: type revolute, parent 3, child 7, origin xyz=-0.4 -0.35 0 rpy=0 0 0, axis 0 1 0, limit lower=-3.14159 upper=3.14159 effort=0.0 velocity=0.0
- added joint 4_6: type revolute, parent 4, child 6, origin xyz=0 0.35 0.35 rpy=0 0 0, axis 0 1 0, limit lower=-3.14159 upper=3.14159 effort=0.0 velocity=0.0
- added joint 7_10: type revolute, parent 7, child 10, origin xyz=0 -0.35 0.4 rpy=0 0 0, axis 0 0 1, limit lower=-3.14159 upper=3.14159 effort=0.0 velocity=0.0
- added joint 8_11: type revolute, parent 8, child 11, origin xyz=0.45 0 0.3 rpy=0 0 0, axis 0 0 1, limit lower=-3.14159 upper=3.14159 effort=0.0 velocity=0.0
- added joint 9_13: type revolute, parent 9, child 13, origin xyz=0 -0.7 0 rpy=0 0 0, axis 0 1 0, limit lower=-3.14159 upper=3.14159 effort=0.0 velocity=0.0
- joint 0_1: axis 1 0 0 -> 0 0 1; origin xyz=0 0.4 0.3 rpy=0 0 0 -> xyz=-0.4 0 0.4 rpy=0 0 0
- joint 0_2: origin xyz=0 0 0.6 rpy=0 0 0 -> xyz=0 0 0.8 rpy=0 0 0

File: body8.urdf (robot description, URDF)
Before this commit: robot robot, 15 links, 14 joints
Links:
- link 0: geometry collision box size=1.0 0.8 0.7; visual box size=1.0 0.8 0.7
- link 1: geometry collision box size=0.6 0.8 0.9; visual box size=0.6 0.8 0.9
- link 10: geometry collision box size=0.7 0.9 1.0; visual box size=0.7 0.9 1.0
- link 11: geometry collision box size=0.7 0.9 0.6; visual box size=0.7 0.9 0.6
- link 12: geometry collision box size=1.0 0.6 0.6; visual box size=1.0 0.6 0.6
- link 13: geometry collision box size=0.8 0.8 0.7; visual box size=0.8 0.8 0.7
- link 14: geometry collision box size=0.6 0.8 0.9; visual box size=0.6 0.8 0.9
- link 2: geometry collision box size=0.6 0.8 0.5; visual box size=0.6 0.8 0.5
- link 3: geometry collision box size=1.0 0.5 0.9; visual box size=1.0 0.5 0.9
- link 4: geometry collision box size=0.6 1.0 0.7; visual box size=0.6 1.0 0.7
- link 5: geometry collision box size=0.9 0.7 0.6; visual box size=0.9 0.7 0.6
- link 6: geometry collision box size=0.8 0.8 0.7; visual box size=0.8 0.8 0.7
- link 7: geometry collision box size=0.8 0.5 0.6; visual box size=0.8 0.5 0.6
- link 8: geometry collision box size=0.8 0.8 0.8; visual box size=0.8 0.8 0.8
- link 9: geometry collision box size=0.6 0.7 0.5; visual box size=0.6 0.7 0.5
Joints:
- removed joint 0_2
- removed joint 10_13
- removed joint 1_10
- removed joint 1_4
- removed joint 2_5
- removed joint 2_7
- removed joint 3_6
- removed joint 4_8
- removed joint 6_9
- removed joint 7_11
- removed joint 8_12
- removed joint 8_14
- added joint 0_4: type revolute, parent 0, child 4, origin xyz=-0.5 0 0.35 rpy=0 0 0, axis 1 0 0, limit lower=-3.14159 upper=3.14159 effort=0.0 velocity=0.0
- added joint 0_9: type revolute, parent 0, child 9, origin xyz=0 -0.4 0.35 rpy=0 0 0, axis 0 0 1, limit lower=-3.14159 upper=3.14159 effort=0.0 velocity=0.0
- added joint 10_12: type revolute, parent 10, child 12, origin xyz=-0.35 0 0.5 rpy=0 0 0, axis 0 1 0, limit lower=-3.14159 upper=3.14159 effort=0.0 velocity=0.0
- added joint 11_13: type revolute, parent 11, child 13, origin xyz=0 -0.9 0 rpy=0 0 0, axis 0 0 1, limit lower=-3.14159 upper=3.14159 effort=0.0 velocity=0.0
- added joint 1_11: type revolute, parent 1, child 11, origin xyz=0 -0.4 0.45 rpy=0 0 0, axis 0 0 1, limit lower=-3.14159 upper=3.14159 effort=0.0 velocity=0.0
- added joint 1_2: type revolute, parent 1, child 2, origin xyz=0 0.4 0.45 rpy=0 0 0, axis 0 1 0, limit lower=-3.14159 upper=3.14159 effort=0.0 velocity=0.0
- added joint 2_8: type revolute, parent 2, child 8, origin xyz=0 0.4 -0.25 rpy=0 0 0, axis 1 0 0, limit lower=-3.14159 upper=3.14159 effort=0.0 velocity=0.0
- added joint 3_14: type revolute, parent 3, child 14, origin xyz=0.5 0 0.45 rpy=0 0 0, axis 0 0 1, limit lower=-3.14159 upper=3.14159 effort=0.0 velocity=0.0
- added joint 3_5: type revolute, parent 3, child 5, origin xyz=0 0 0.9 rpy=0 0 0, axis 0 0 1, limit lower=-3.14159 upper=3.14159 effort=0.0 velocity=0.0
- added joint 4_10: type revolute, parent 4, child 10, origin xyz=-0.3 0 0.35 rpy=0 0 0, axis 1 0 0, limit lower=-3.14159 upper=3.14159 effort=0.0 velocity=0.0
- added joint 4_6: type revolute, parent 4, child 6, origin xyz=-0.3 0.5 0 rpy=0 0 0, axis 0 0 1, limit lower=-3.14159 upper=3.14159 effort=0.0 velocity=0.0
- added joint 5_7: type revolute, parent 5, child 7, origin xyz=-0.45 0 0.3 rpy=0 0 0, axis 0 0 1, limit lower=-3.14159 upper=3.14159 effort=0.0 velocity=0.0
- joint 0_1: axis 1 0 0 -> 0 0 1; origin xyz=0 0.4 0.3 rpy=0 0 0 -> xyz=0 0 0.7 rpy=0 0 0
- joint 2_3: origin xyz=0.45 0 0.35 rpy=0 0 0 -> xyz=0 0.4 0.25 rpy=0 0 0

File: body9.urdf (robot description, URDF)
Before this commit: robot robot, 15 links, 14 joints
Links:
- link 0: geometry collision box size=0.7 1.0 0.5; visual box size=0.7 1.0 0.5
- link 1: geometry collision box size=0.7 0.8 1.0; visual box size=0.7 0.8 1.0
- link 10: geometry collision box size=0.6 0.5 0.5; visual box size=0.6 0.5 0.5
- link 11: geometry collision box size=0.9 0.8 0.9; visual box size=0.9 0.8 0.9
- link 12: geometry collision box size=0.7 0.7 0.5; visual box size=0.7 0.7 0.5
- link 13: geometry collision box size=0.7 0.8 0.6; visual box size=0.7 0.8 0.6
- link 14: geometry collision box size=0.5 1.0 0.5; visual box size=0.5 1.0 0.5
- link 2: geometry collision box size=1.0 0.6 0.7; visual box size=1.0 0.6 0.7
- link 3: geometry collision box size=0.6 0.5 1.0; visual box size=0.6 0.5 1.0
- link 4: geometry collision box size=0.6 0.9 0.6; visual box size=0.6 0.9 0.6
- link 5: geometry collision box size=0.7 0.9 0.9; visual box size=0.7 0.9 0.9
- link 6: geometry collision box size=0.7 0.9 0.7; visual box size=0.7 0.9 0.7
- link 7: geometry collision box size=0.8 0.8 0.5; visual box size=0.8 0.8 0.5
- link 8: geometry collision box size=0.7 0.6 0.6; visual box size=0.7 0.6 0.6
- link 9: geometry collision box size=0.8 0.5 0.6; visual box size=0.8 0.5 0.6
Joints:
- removed joint 0_2
- removed joint 10_13
- removed joint 1_10
- removed joint 1_4
- removed joint 2_3
- removed joint 2_5
- removed joint 2_7
- removed joint 3_6
- removed joint 4_8
- removed joint 6_9
- removed joint 7_11
- removed joint 8_12
- removed joint 8_14
- added joint 0_7: type revolute, parent 0, child 7, origin xyz=0.35 0 0.25 rpy=0 0 0, axis 0 1 0, limit lower=-3.14159 upper=3.14159 effort=0.0 velocity=0.0
- added joint 12_14: type revolute, parent 12, child 14, origin xyz=0.35 0 0.25 rpy=0 0 0, axis 0 1 0, limit lower=-3.14159 upper=3.14159 effort=0.0 velocity=0.0
- added joint 1_2: type revolute, parent 1, child 2, origin xyz=0 0 1.0 rpy=0 0 0, axis 1 0 0, limit lower=-3.14159 upper=3.14159 effort=0.0 velocity=0.0
- added joint 1_3: type revolute, parent 1, child 3, origin xyz=0 0.4 0.5 rpy=0 0 0, axis 0 1 0, limit lower=-3.14159 upper=3.14159 effort=0.0 velocity=0.0
- added joint 1_5: type revolute, parent 1, child 5, origin xyz=-0.35 0 0.5 rpy=0 0 0, axis 0 0 1, limit lower=-3.14159 upper=3.14159 effort=0.0 velocity=0.0
- added joint 1_6: type revolute, parent 1, child 6, origin xyz=0.35 0 0.5 rpy=0 0 0, axis 0 0 1, limit lower=-3.14159 upper=3.14159 effort=0.0 velocity=0.0
- added joint 2_4: type revolute, parent 2, child 4, origin xyz=0 0.3 0.35 rpy=0 0 0, axis 0 1 0, limit lower=-3.14159 upper=3.14159 effort=0.0 velocity=0.0
- added joint 2_8: type revolute, parent 2, child 8, origin xyz=0 0 0.7 rpy=0 0 0, axis 0 1 0, limit lower=-3.14159 upper=3.14159 effort=0.0 velocity=0.0
- added joint 3_13: type revolute, parent 3, child 13, origin xyz=0 0.5 0 rpy=0 0 0, axis 0 1 0, limit lower=-3.14159 upper=3.14159 effort=0.0 velocity=0.0
- added joint 4_9: type revolute, parent 4, child 9, origin xyz=0 0.45 0.3 rpy=0 0 0, axis 0 0 1, limit lower=-3.14159 upper=3.14159 effort=0.0 velocity=0.0
- added joint 6_11: type revolute, parent 6, child 11, origin xyz=0.35 -0.45 0 rpy=0 0 0, axis 0 1 0, limit lower=-3.14159 upper=3.14159 effort=0.0 velocity=0.0
- added joint 6_12: type revolute, parent 6, child 12, origin xyz=0.7 0 0 rpy=0 0 0, axis 1 0 0, limit lower=-3.14159 upper=3.14159 effort=0.0 velocity=0.0
- added joint 9_10: type revolute, parent 9, child 10, origin xyz=0 0.25 0.3 rpy=0 0 0, axis 0 0 1, limit lower=-3.14159 upper=3.14159 effort=0.0 velocity=0.0
- joint 0_1: origin xyz=0 0.4 0.3 rpy=0 0 0 -> xyz=0 0 0.5 rpy=0 0 0
