Commit message: done

File: bestineachseed/body_seed0.urdf (robot description, URDF)
Before this commit: robot robot, 9 links, 8 joints
Links:
- removed link 8
- link 0: geometry collision box size=0.7 0.9 1.0; visual box size=0.7 0.9 1.0
- link 1: geometry collision box size=0.5 0.5 0.9; visual box size=0.5 0.5 0.9
- link 2: geometry collision box size=0.7 0.8 0.7; visual box size=0.7 0.8 0.7
- link 3: geometry collision box size=0.6 0.8 0.9; visual box size=0.6 0.8 0.9
- link 4: geometry collision box size=0.9 0.7 0.6; visual box size=0.9 0.7 0.6
- link 5: geometry collision box size=0.7 1.0 0.5; visual box size=0.7 1.0 0.5
- link 6: geometry collision box size=0.8 0.6 0.5; visual box size=0.8 0.6 0.5
- link 7: geometry collision box size=0.5 0.7 1.0; visual box size=0.5 0.7 1.0
Joints:
- removed joint 0_5
- removed joint 0_6
- removed joint 1_2
- removed joint 7_8
- added joint 0_2: type revolute, parent 0, child 2, origin xyz=-0.35 0 0.5 rpy=0 0 0, axis 0 0 1, limit lower=-3.14159 upper=3.14159 effort=0.0 velocity=0.0
- added joint 1_6: type revolute, parent 1, child 6, origin xyz=0.5 0 0 rpy=0 0 0, axis 0 0 1, limit lower=-3.14159 upper=3.14159 effort=0.0 velocity=0.0
- added joint 3_5: type revolute, parent 3, child 5, origin xyz=0 0.4 0.45 rpy=0 0 0, axis 0 0 1, limit lower=-3.14159 upper=3.14159 effort=0.0 velocity=0.0
- joint 0_1: origin xyz=0 0.4 0.4 rpy=0 0 0 -> xyz=0.35 0 0.5 rpy=0 0 0
- joint 2_3: axis 0 0 1 -> 1 0 0; origin xyz=0.25 0.4 0 rpy=0 0 0 -> xyz=-0.35 0.4 0 rpy=0 0 0
- joint 3_4: axis 1 0 0 -> 0 1 0; origin xyz=0 0.25 0.25 rpy=0 0 0 -> xyz=-0.3 0.4 0 rpy=0 0 0
- joint 5_7: axis 1 0 0 -> 0 1 0; origin xyz=-0.4 0 0.3 rpy=0 0 0 -> xyz=0.35 0 0.25 rpy=0 0 0

File: bestineachseed/body_seed1.urdf (robot description, URDF)
Before this commit: robot robot, 12 links, 11 joints
Links:
- added link 12, mass 1; collision box size=0.6 0.8 0.6; visual box size=0.6 0.8 0.6
- link 0: geometry collision box size=0.9 0.8 0.7; visual box size=0.9 0.8 0.7
- link 1: geometry collision box size=0.6 0.8 0.5; visual box size=0.6 0.8 0.5
- link 10: geometry collision box size=0.6 0.6 1.0; visual box size=0.6 0.6 1.0
- link 11: geometry collision box size=1.0 0.8 0.6; visual box size=1.0 0.8 0.6
- link 2: geometry collision box size=0.9 0.7 0.8; visual box size=0.9 0.7 0.8
- link 3: geometry collision box size=0.8 0.7 0.6; visual box size=0.8 0.7 0.6
- link 4: geometry collision box size=0.9 0.9 1.0; visual box size=0.9 0.9 1.0
- link 5: geometry collision box size=0.5 0.6 0.6; visual box size=0.5 0.6 0.6
- link 6: geometry collision box size=0.6 0.6 1.0; visual box size=0.6 0.6 1.0
- link 7: geometry collision box size=0.8 0.6 0.6; visual box size=0.8 0.6 0.6
- link 8: geometry collision box size=0.5 0.5 0.9; visual box size=0.5 0.5 0.9
- link 9: geometry collision box size=0.6 0.8 0.7; visual box size=0.6 0.8 0.7
Joints:
- removed joint 0_3
- removed joint 0_7
- removed joint 2_5
- removed joint 2_8
- removed joint 2_9
- removed joint 4_11
- removed joint 9_10
- added joint 0_9: type revolute, parent 0, child 9, origin xyz=0 -0.4 0.35 rpy=0 0 0, axis 1 0 0, limit lower=-3.14159 upper=3.14159 effort=0.0 velocity=0.0
- added joint 2_10: type revolute, parent 2, child 10, origin xyz=-0.45 0 0.4 rpy=0 0 0, axis 0 1 0, limit lower=-3.14159 upper=3.14159 effort=0.0 velocity=0.0
- added joint 2_3: type revolute, parent 2, child 3, origin xyz=0 0.35 0.4 rpy=0 0 0, axis 0 0 1, limit lower=-3.14159 upper=3.14159 effort=0.0 velocity=0.0
- added joint 3_8: type revolute, parent 3, child 8, origin xyz=-0.4 0.35 0 rpy=0 0 0, axis 0 1 0, limit lower=-3.14159 upper=3.14159 effort=0.0 velocity=0.0
- added joint 4_12: type revolute, parent 4, child 12, origin xyz=0 0.9 0 rpy=0 0 0, axis 1 0 0, limit lower=-3.14159 upper=3.14159 effort=0.0 velocity=0.0
- added joint 4_5: type revolute, parent 4, child 5, origin xyz=0 0.45 0.5 rpy=0 0 0, axis 1 0 0, limit lower=-3.14159 upper=3.14159 effort=0.0 velocity=0.0
- added joint 4_7: type revolute, parent 4, child 7, origin xyz=-0.45 0.45 0 rpy=0 0 0, axis 0 1 0, limit lower=-3.14159 upper=3.14159 effort=0.0 velocity=0.0
- added joint 5_11: type revolute, parent 5, child 11, origin xyz=-0.25 0 0.3 rpy=0 0 0, axis 1 0 0, limit lower=-3.14159 upper=3.14159 effort=0.0 velocity=0.0
- joint 0_1: axis 0 0 1 -> 0 1 0; origin xyz=0.35 0 0.45 rpy=0 0 0 -> xyz=0 0.4 0.35 rpy=0 0 0
- joint 0_2: axis 0 0 1 -> 0 1 0; origin xyz=-0.35 0 0.45 rpy=0 0 0 -> xyz=0 0 0.7 rpy=0 0 0
- joint 3_4: axis 1 0 0 -> 0 1 0; origin xyz=0.35 -0.45 0 rpy=0 0 0 -> xyz=0 0.7 0 rpy=0 0 0
- joint 3_6: origin xyz=0 -0.45 0.3 rpy=0 0 0 -> xyz=0 0.35 0.3 rpy=0 0 0

File: bestineachseed/body_seed2.urdf (robot description, URDF)
Before this commit: robot robot, 5 links, 4 joints
Links:
- link 0: geometry collision box size=0.7 0.7 0.5; visual box size=0.7 0.7 0.5
- link 1: geometry collision box size=1.0 0.9 0.6; visual box size=1.0 0.9 0.6
- link 2: geometry collision box size=1.0 0.6 0.8; visual box size=1.0 0.6 0.8
- link 3: geometry collision box size=0.6 0.6 0.7; visual box size=0.6 0.6 0.7
- link 4: geometry collision box size=0.6 0.8 0.6; visual box size=0.6 0.8 0.6
Joints:
- removed joint 0_4
- added joint 3_4: type revolute, parent 3, child 4, origin xyz=0.3 0 0.35 rpy=0 0 0, axis 1 0 0, limit lower=-3.14159 upper=3.14159 effort=0.0 velocity=0.0
- joint 0_1: axis 0 1 0 -> 1 0 0; origin xyz=-0.4 0 0.3 rpy=0 0 0 -> xyz=0 0 0.5 rpy=0 0 0
- joint 1_2: axis 0 0 1 -> 0 1 0; origin xyz=-0.5 0 0 rpy=0 0 0 -> xyz=-0.5 0 0.3 rpy=0 0 0
- joint 2_3: axis 1 0 0 -> 0 0 1; origin xyz=-0.3 0 0.3 rpy=0 0 0 -> xyz=-0.5 0 0.4 rpy=0 0 0

File: bestineachseed/body_seed3.urdf (robot description, URDF)
Before this commit: robot robot, 11 links, 10 joints
Links:
- removed link 10
- removed link 9
- link 0: geometry collision box size=0.6 0.9 1.0; visual box size=0.6 0.9 1.0
- link 1: geometry collision box size=0.6 0.6 0.7; visual box size=0.6 0.6 0.7
- link 2: geometry collision box size=0.9 0.6 0.5; visual box size=0.9 0.6 0.5
- link 3: geometry collision box size=0.7 0.9 0.6; visual box size=0.7 0.9 0.6
- link 4: geometry collision box size=1.0 0.6 0.9; visual box size=1.0 0.6 0.9
- link 5: geometry collision box size=0.8 0.8 0.7; visual box size=0.8 0.8 0.7
- link 6: geometry collision box size=0.6 0.8 0.6; visual box size=0.6 0.8 0.6
- link 7: geometry collision box size=0.6 0.6 1.0; visual box size=0.6 0.6 1.0
- link 8: geometry collision box size=0.6 0.5 0.8; visual box size=0.6 0.5 0.8
Joints:
- removed joint 1_2
- removed joint 1_4
- removed joint 1_9
- removed joint 3_7
- removed joint 4_5
- removed joint 6_10
- removed joint 7_8
- added joint 0_2: type revolute, parent 0, child 2, origin xyz=0 0.45 0.5 rpy=0 0 0, axis 1 0 0, limit lower=-3.14159 upper=3.14159 effort=0.0 velocity=0.0
- added joint 1_7: type revolute, parent 1, child 7, origin xyz=-0.3 -0.3 0 rpy=0 0 0, axis 1 0 0, limit lower=-3.14159 upper=3.14159 effort=0.0 velocity=0.0
- added joint 2_4: type revolute, parent 2, child 4, origin xyz=0 0.6 0 rpy=0 0 0, axis 0 0 1, limit lower=-3.14159 upper=3.14159 effort=0.0 velocity=0.0
- added joint 3_5: type revolute, parent 3, child 5, origin xyz=0 0.45 0.3 rpy=0 0 0, axis 1 0 0, limit lower=-3.14159 upper=3.14159 effort=0.0 velocity=0.0
- added joint 6_8: type revolute, parent 6, child 8, origin xyz=0.3 -0.4 0 rpy=0 0 0, axis 1 0 0, limit lower=-3.14159 upper=3.14159 effort=0.0 velocity=0.0
- joint 0_1: axis 1 0 0 -> 0 1 0; origin xyz=0 -0.45 0.35 rpy=0 0 0 -> xyz=0 -0.45 0.5 rpy=0 0 0
- joint 0_3: axis 0 1 0 -> 1 0 0; origin xyz=0 0.45 0.35 rpy=0 0 0 -> xyz=0 0 1.0 rpy=0 0 0
- joint 0_6: origin xyz=0.4 0 0.35 rpy=0 0 0 -> xyz=0.3 0 0.5 rpy=0 0 0

File: bestineachseed/body_seed4.urdf (robot description, URDF)
Before this commit: robot robot, 6 links, 5 joints
Links:
- added link 6, mass 1; collision box size=0.6 0.6 0.6; visual box size=0.6 0.6 0.6
- link 0: geometry collision box size=0.7 0.6 0.8; visual box size=0.7 0.6 0.8
- link 1: geometry collision box size=0.8 0.9 0.6; visual box size=0.8 0.9 0.6
- link 2: geometry collision box size=0.5 0.6 0.5; visual box size=0.5 0.6 0.5
- link 3: geometry collision box size=0.8 0.6 0.8; visual box size=0.8 0.6 0.8
- link 4: geometry collision box size=0.7 0.7 0.5; visual box size=0.7 0.7 0.5
- link 5: geometry collision box size=0.9 0.6 0.7; visual box size=0.9 0.6 0.7
Joints:
- removed joint 0_2
- removed joint 2_3
- removed joint 3_5
- added joint 1_2: type revolute, parent 1, child 2, origin xyz=0 0.9 0 rpy=0 0 0, axis 0 1 0, limit lower=-3.14159 upper=3.14159 effort=0.0 velocity=0.0
- added joint 1_3: type revolute, parent 1, child 3, origin xyz=0.4 0.45 0 rpy=0 0 0, axis 0 1 0, limit lower=-3.14159 upper=3.14159 effort=0.0 velocity=0.0
- added joint 2_5: type revolute, parent 2, child 5, origin xyz=0 0.3 0.25 rpy=0 0 0, axis 0 0 1, limit lower=-3.14159 upper=3.14159 effort=0.0 velocity=0.0
- added joint 5_6: type revolute, parent 5, child 6, origin xyz=0.45 0 0.35 rpy=0 0 0, axis 1 0 0, limit lower=-3.14159 upper=3.14159 effort=0.0 velocity=0.0
- joint 0_1: axis 0 1 0 -> 1 0 0; origin xyz=-0.3 0 0.3 rpy=0 0 0 -> xyz=0 0.3 0.4 rpy=0 0 0
- joint 0_4: axis 1 0 0 -> 0 1 0; origin xyz=0 -0.45 0.3 rpy=0 0 0 -> xyz=0 0 0.8 rpy=0 0 0

File: body11.urdf (robot description, URDF)
Before this commit: robot robot, 8 links, 7 joints
Links:
- added link 10, mass 1; collision box size=0.6 0.6 1.0; visual box size=0.6 0.6 1.0
- added link 11, mass 1; collision box size=1.0 0.8 0.6; visual box size=1.0 0.8 0.6
- added link 12, mass 1; collision box size=0.6 0.8 0.6; visual box size=0.6 0.8 0.6
- added link 8, mass 1; collision box size=0.5 0.5 0.9; visual box size=0.5 0.5 0.9
- added link 9, mass 1; collision box size=0.6 0.8 0.7; visual box size=0.6 0.8 0.7
- link 0: geometry collision box size=0.9 0.8 0.7; visual box size=0.9 0.8 0.7
- link 1: geometry collision box size=0.6 0.8 0.5; visual box size=0.6 0.8 0.5
- link 2: geometry collision box size=0.9 0.7 0.8; visual box size=0.9 0.7 0.8
- link 3: geometry collision box size=0.8 0.7 0.6; visual box size=0.8 0.7 0.6
- link 4: geometry collision box size=0.9 0.9 1.0; visual box size=0.9 0.9 1.0
- link 5: geometry collision box size=0.5 0.6 0.6; visual box size=0.5 0.6 0.6
- link 6: geometry collision box size=0.6 0.6 1.0; visual box size=0.6 0.6 1.0
- link 7: geometry collision box size=0.8 0.6 0.6; visual box size=0.8 0.6 0.6
Joints:
- removed joint 1_6
- removed joint 3_5
- removed joint 5_7
- added joint 0_9: type revolute, parent 0, child 9, origin xyz=0 -0.4 0.35 rpy=0 0 0, axis 1 0 0, limit lower=-3.14159 upper=3.14159 effort=0.0 velocity=0.0
- added joint 2_10: type revolute, parent 2, child 10, origin xyz=-0.45 0 0.4 rpy=0 0 0, axis 0 1 0, limit lower=-3.14159 upper=3.14159 effort=0.0 velocity=0.0
- added joint 3_6: type revolute, parent 3, child 6, origin xyz=0 0.35 0.3 rpy=0 0 0, axis 0 0 1, limit lower=-3.14159 upper=3.14159 effort=0.0 velocity=0.0
- added joint 3_8: type revolute, parent 3, child 8, origin xyz=-0.4 0.35 0 rpy=0 0 0, axis 0 1 0, limit lower=-3.14159 upper=3.14159 effort=0.0 velocity=0.0
- added joint 4_12: type revolute, parent 4, child 12, origin xyz=0 0.9 0 rpy=0 0 0, axis 1 0 0, limit lower=-3.14159 upper=3.14159 effort=0.0 velocity=0.0
- added joint 4_5: type revolute, parent 4, child 5, origin xyz=0 0.45 0.5 rpy=0 0 0, axis 1 0 0, limit lower=-3.14159 upper=3.14159 effort=0.0 velocity=0.0
- added joint 4_7: type revolute, parent 4, child 7, origin xyz=-0.45 0.45 0 rpy=0 0 0, axis 0 1 0, limit lower=-3.14159 upper=3.14159 effort=0.0 velocity=0.0
- added joint 5_11: type revolute, parent 5, child 11, origin xyz=-0.25 0 0.3 rpy=0 0 0, axis 1 0 0, limit lower=-3.14159 upper=3.14159 effort=0.0 velocity=0.0
- joint 0_1: axis 0 0 1 -> 0 1 0; origin xyz=0.35 0 0.5 rpy=0 0 0 -> xyz=0 0.4 0.35 rpy=0 0 0
- joint 0_2: axis 0 0 1 -> 0 1 0; origin xyz=-0.35 0 0.5 rpy=0 0 0 -> xyz=0 0 0.7 rpy=0 0 0
- joint 2_3: axis 1 0 0 -> 0 0 1; origin xyz=-0.35 0.4 0 rpy=0 0 0 -> xyz=0 0.35 0.4 rpy=0 0 0
- joint 3_4: origin xyz=-0.3 0.4 0 rpy=0 0 0 -> xyz=0 0.7 0 rpy=0 0 0

File: body111.urdf (robot description, URDF)
Before this commit: robot robot, 10 links, 9 joints
Links:
- removed link 9
- link 0: geometry collision box size=0.6 0.9 1.0; visual box size=0.6 0.9 1.0
- link 1: geometry collision box size=0.6 0.6 0.7; visual box size=0.6 0.6 0.7
- link 2: geometry collision box size=0.9 0.6 0.5; visual box size=0.9 0.6 0.5
- link 3: geometry collision box size=0.7 0.9 0.6; visual box size=0.7 0.9 0.6
- link 4: geometry collision box size=1.0 0.6 0.9; visual box size=1.0 0.6 0.9
- link 5: geometry collision box size=0.8 0.8 0.7; visual box size=0.8 0.8 0.7
- link 6: geometry collision box size=0.6 0.8 0.6; visual box size=0.6 0.8 0.6
- link 7: geometry collision box size=0.6 0.6 1.0; visual box size=0.6 0.6 1.0
- link 8: geometry collision box size=0.6 0.5 0.8; visual box size=0.6 0.5 0.8
Joints:
- removed joint 1_2
- removed joint 1_4
- removed joint 1_6
- removed joint 2_3
- removed joint 2_8
- removed joint 4_7
- removed joint 7_9
- added joint 0_2: type revolute, parent 0, child 2, origin xyz=0 0.45 0.5 rpy=0 0 0, axis 1 0 0, limit lower=-3.14159 upper=3.14159 effort=0.0 velocity=0.0
- added joint 0_3: type revolute, parent 0, child 3, origin xyz=0 0 1.0 rpy=0 0 0, axis 1 0 0, limit lower=-3.14159 upper=3.14159 effort=0.0 velocity=0.0
- added joint 0_6: type revolute, parent 0, child 6, origin xyz=0.3 0 0.5 rpy=0 0 0, axis 0 0 1, limit lower=-3.14159 upper=3.14159 effort=0.0 velocity=0.0
- added joint 1_7: type revolute, parent 1, child 7, origin xyz=-0.3 -0.3 0 rpy=0 0 0, axis 1 0 0, limit lower=-3.14159 upper=3.14159 effort=0.0 velocity=0.0
- added joint 2_4: type revolute, parent 2, child 4, origin xyz=0 0.6 0 rpy=0 0 0, axis 0 0 1, limit lower=-3.14159 upper=3.14159 effort=0.0 velocity=0.0
- added joint 6_8: type revolute, parent 6, child 8, origin xyz=0.3 -0.4 0 rpy=0 0 0, axis 1 0 0, limit lower=-3.14159 upper=3.14159 effort=0.0 velocity=0.0
- joint 0_1: origin xyz=0 0 1.0 rpy=0 0 0 -> xyz=0 -0.45 0.5 rpy=0 0 0
- joint 3_5: origin xyz=0 0.5 0.3 rpy=0 0 0 -> xyz=0 0.45 0.3 rpy=0 0 0

File: body1111.urdf (robot description, URDF)
Before this commit: robot robot, 5 links, 4 joints
Links:
- link 0: geometry collision box size=0.7 0.7 0.5; visual box size=0.7 0.7 0.5
- link 1: geometry collision box size=1.0 0.9 0.6; visual box size=1.0 0.9 0.6
- link 2: geometry collision box size=1.0 0.6 0.8; visual box size=1.0 0.6 0.8
- link 3: geometry collision box size=0.6 0.6 0.7; visual box size=0.6 0.6 0.7
- link 4: geometry collision box size=0.6 0.8 0.6; visual box size=0.6 0.8 0.6
Joints:
- removed joint 0_2
- added joint 1_2: type revolute, parent 1, child 2, origin xyz=-0.5 0 0.3 rpy=0 0 0, axis 0 1 0, limit lower=-3.14159 upper=3.14159 effort=0.0 velocity=0.0
- joint 0_1: axis 0 1 0 -> 1 0 0; origin xyz=0 0 0.9 rpy=0 0 0 -> xyz=0 0 0.5 rpy=0 0 0
- joint 2_3: axis 0 1 0 -> 0 0 1; origin xyz=0.45 0 0.4 rpy=0 0 0 -> xyz=-0.5 0 0.4 rpy=0 0 0
- joint 3_4: axis 0 1 0 -> 1 0 0; origin xyz=0 0 0.9 rpy=0 0 0 -> xyz=0.3 0 0.35 rpy=0 0 0
